Commit message: cleaned urdf and rviz

File: urdf/pendulum.urdf (robot description, URDF)
Before this commit: robot pendulum, 3 links, 2 joints
Links:
- link pendulum_link: geometry collision sphere radius=0.08; visual sphere radius=0.08
- link pendulum_rod_link: geometry collision cylinder length=2 radius=0.1; visual cylinder length=2 radius=0.02
