Commit message: fixed a bug in water_current calculatoins

File: urdf/pendulum.urdf.xacro (robot description, xacro)
@@ -4,7 +4,7 @@
 <xacro:property name="params" value="${load_yaml(yaml_file)}"/>
 <xacro:property name="radius" value="${params[Link1][val1]}" /> -->
- <xacro:property name="radius" value="0.5" />
-<xacro:property name="length" value="5.0" />
-<xacro:property name="rod_radius" value="0.05" />
+ <xacro:property name="radius" value="0.1" />
+<xacro:property name="length" value="2.0" />
+<xacro:property name="rod_radius" value="0.01" />
     <joint name="pendulum_joint" type="continuous">
       <origin xyz="0 0 0" rpy="0 1.57 0 "/>
